Commit message: script cleaned

File: urdf/robot.urdf.xacro (robot description, xacro)
@@ -3,9 +3,9 @@
   <link name="base_link">
     <visual>
-      <geometry><cylinder radius="0.035" length="0.05"/></geometry>
+      <geometry><cylinder radius="0.071" length="0.05"/></geometry>
       <material name="blue"><color rgba="0 0 1 1"/></material>
     </visual>
     <collision>
-      <geometry><cylinder radius="0.035" length="0.05"/></geometry>
+      <geometry><cylinder radius="0.071" length="0.05"/></geometry>
     </collision>
     <inertial>
