Commit message: sph fixed

File: install/SPH/share/SPH/urdf/robot.urdf.xacro (robot description, xacro)
@@ -1 +1,53 @@
-/home/azivinicius/ros2_ws/src/SPH/build/SPH/urdf/robot.urdf.xacro
+<?xml version="1.0"?>
+<robot xmlns:xacro="http://www.ros.org/wiki/xacro" name="diff_robot">
+  <link name="base_link">
+    <visual>
+      <geometry><cylinder radius="0.071" length="0.05"/></geometry>
+      <material name="blue"><color rgba="0 0 1 1"/></material>
+    </visual>
+    <collision>
+      <geometry><cylinder radius="0.071" length="0.05"/></geometry>
+    </collision>
+    <inertial>
+      <mass value="1.0"/>
+      <inertia ixx="0.005" ixy="0" ixz="0" iyy="0.005" iyz="0" izz="0.005"/>
+    </inertial>
+  </link>
+  <link name="left_wheel">
+    <visual><geometry><cylinder radius="0.033" length="0.018"/></geometry></visual>
+    <collision><geometry><cylinder radius="0.033" length="0.018"/></geometry></collision>
+    <inertial>
+      <mass value="0.1"/>
+      <inertia ixx="0.0001" ixy="0" ixz="0" iyy="0.0001" iyz="0" izz="0.0001"/>
+    </inertial>
+  </link>
+  <link name="right_wheel">
+    <visual><geometry><cylinder radius="0.033" length="0.018"/></geometry></visual>
+    <collision><geometry><cylinder radius="0.033" length="0.018"/></geometry></collision>
+    <inertial>
+      <mass value="0.1"/>
+      <inertia ixx="0.0001" ixy="0" ixz="0" iyy="0.0001" iyz="0" izz="0.0001"/>
+    </inertial>
+  </link>
+  <joint name="left_wheel_joint" type="continuous">
+    <parent link="base_link"/><child link="left_wheel"/>
+    <origin xyz="0 0.08 0" rpy="-1.57 0 0"/><axis xyz="0 0 1"/>
+  </joint>
+  <joint name="right_wheel_joint" type="continuous">
+    <parent link="base_link"/><child link="right_wheel"/>
+    <origin xyz="0 -0.08 0" rpy="-1.57 0 0"/><axis xyz="0 0 1"/>
+  </joint>
+  <gazebo>
+    <plugin filename="gz-sim-diff-drive-system" name="gz::sim::systems::DiffDrive">
+      <left_joint>left_wheel_joint</left_joint>
+      <right_joint>right_wheel_joint</right_joint>
+      <wheel_separation>0.16</wheel_separation>
+      <wheel_radius>0.033</wheel_radius>
+      <odom_publish_frequency>50</odom_publish_frequency>
+      <topic>cmd_vel</topic>
+      <odom_topic>odom</odom_topic>
+      <frame_id>odom</frame_id>
+      <child_frame_id>base_link</child_frame_id>
+    </plugin>
+  </gazebo>
+</robot>

File: urdf/robot.urdf.xacro (robot description, xacro)
@@ -1,4 +1,6 @@
 <?xml version="1.0"?>
 <robot xmlns:xacro="http://www.ros.org/wiki/xacro" name="diff_robot">
+<xacro:arg name="robot_name" default="robot_0"/>
+<xacro:property name="ns" value="$(arg robot_name)"/>
   <link name="base_link">
     <visual>
@@ -45,8 +47,10 @@
       <wheel_radius>0.033</wheel_radius>
       <odom_publish_frequency>50</odom_publish_frequency>
-      <topic>cmd_vel</topic>
-      <odom_topic>odom</odom_topic>
-      <frame_id>odom</frame_id>
-      <child_frame_id>base_link</child_frame_id>
+      <!-- 2. FORCE O TOPICO A USAR O NAMESPACE DO ROBÔ -->
+      <topic>/${ns}/cmd_vel</topic>
+      <odom_topic>/${ns}/odom</odom_topic>
+      <!-- 3. AJUSTE OS FRAMES PARA REBATER O NAMESPACE (Evita TF duplicado) -->
+      <frame_id>${ns}/odom</frame_id>
+      <child_frame_id>${ns}/base_link</child_frame_id>
     </plugin>
   </gazebo>
